File: layout/cnode_rev_a.sch (EAGLE design)
At the start: 40 parts, among them IC1 LPC1347TQFP48, IC2 MCP1755-SOT23-5, IC3 DWM1000, IC4 MPU-9250, Q1 BC807-16SMD, X1 MINI-USB-SCHIELD-32005-201, Y1 MT-CRYSTAL 12MHz

Commit message: Updated to STM32-based node for ATLAS 2.0 release
Parts:
- removed C10, C8, C9: 100nF, rcl:C-EUC0603
- removed C11: 10µF, rcl:C-EUC0603
- removed IC3: DWM1000, decawave:DWM1000
- removed IC4: MPU-9250, invensense:MPU-9250
- removed JP1: (no value), microbuilder:HEADER-1X4ROUND
- removed JTAG: (no value), nxp:ARM-JTAG_1.27-SMD
- removed L1: EMI, rcl:R-EU_R0603
- removed Q1: BC807-16SMD, transistor-pnp:BC807-16SMD
- removed R10, R11, R13: 1k, rcl:R-EU_R0603
- removed R8: 100k, rcl:R-EU_R0603
- removed R9: 10k, rcl:R-EU_R0603
- removed SCL, SDA: (no value), microbuilder:HEADER-1X12MM
- removed SYNC: U.FL, microbuilder:U.FL
- removed U$1: TACT-SWITCH-40-40, tactile-switch:TACT-SWITCH-40-40
- removed X1: MINI-USB-SCHIELD-32005-201, con-cypressindustries:MINI-USB-SCHIELD-32005-201
- removed Y1: MT-CRYSTAL 12MHz, euroquartz:MT-CRYSTAL
- added ACT: White, microbuilder:LED0805_NOOUTLINE
- added BOARD1: STM32F103C8T6BOARD, stm32board:STM32F103C8T6BOARD
- added CN_IMU: (no value), microbuilder:HEADER-1X10ROUND
- added CN_USART1, CN_USART2: (no value), microbuilder:HEADER-1X3ROUND
- added ERR: Red, microbuilder:LED0805_NOOUTLINE
- added OK: Green, microbuilder:LED0805_NOOUTLINE
- added SFD: Yellow, microbuilder:LED0805_NOOUTLINE
- C1, C2: value 18p -> 22uF; device rcl:C-EUC0603 -> rcl:C-EUC0805
- C3: value 10nF -> 22uF; device rcl:C-EUC0603 -> rcl:C-EUC0805
- C4: value 100nF -> 22uF; device rcl:C-EUC0603 -> rcl:C-EUC0805
- C5, C6: value 10µF/6.3V -> 10uF; device rcl:C-EUC0603 -> rcl:C-EUC0805
- C7: value 10nF -> 470pF; device rcl:C-EUC0603 -> rcl:C-EUC0805
- IC1: value LPC1347TQFP48 -> DWM1000; device lpc1xxx:LPC1347TQFP48 -> decawave:DWM1000
- IC2: value MCP1755-SOT23-5 -> MIC5219-3.3; device vreg:LP2985-SOT23-5 -> v-reg-micrel:MIC5219XX
- R1, R2: value 33R -> 1k; device rcl:R-EU_R0603 -> rcl:R-EU_R0805
- R3, R5: device rcl:R-EU_R0603 -> rcl:R-EU_R0805
- R4, R6, R7: value 10k -> 1k; device rcl:R-EU_R0603 -> rcl:R-EU_R0805
- RX: value (none) -> Green; device led:LEDCHIP-LED0603 -> microbuilder:LED0805_NOOUTLINE
- SYS: value (none) -> White; device led:LEDCHIP-LED0603 -> microbuilder:LED0805_NOOUTLINE
- TX: value (none) -> Red; device led:LEDCHIP-LED0603 -> microbuilder:LED0805_NOOUTLINE
Connections:
- removed net +5V: C5.1, IC2.IN, IC2.ON/!OFF, L1.1, R9.2
- removed net JTAG_RTCK: JTAG.7
- removed net JTAG_SWCLK: IC1.SWCLK/PIO0_10/SCK0/CT16B0_MAT2, JTAG.4
- removed net JTAG_SWDIO: IC1.SWDIO/PIO0_15/AD4/CT32B1_MAT2, JTAG.2
- removed net JTAG_SWI: JTAG.8
- removed net JTAG_SWO: IC1.PIO0_9/MOSI0/CT16B0_MAT1/SWO, JTAG.6
- removed net LED_OK: IC3.GPIO0/RXOKLED
- removed net N$10: R11.1, RX.A
- removed net N$11: R13.1, SYS.A
- removed net N$12: C3.1, IC4.REGOUT
- removed net N$20: C7.1, IC2.NC/FB
- removed net N$28: JTAG.1
- removed net N$36: R2.2, R3.2, X1G$1.3
- removed net RESET: IC1.RESET/PIO0_0, JTAG.10, U$1.P$2
- removed net SCL: IC1.PIO0_4/SCL, IC4.SCL/SCLK, R7.2, SCL.1
- removed net SDA: IC1.PIO0_5/SDA, IC4.SDA/SDI, R6.2, SDA.1
- removed net SPI1_SSEL: IC1.PIO1_19/DTR/SSEL1, IC3.!SPICS
- removed net USART1_RXD: IC1.PIO1_14/DSR/CT16B0_MAT1/RXD, JP1.3
- removed net USART1_TXD: IC1.PIO1_13/DTR/CT16B0_MAT0/TXD, JP1.2
- removed net USB_CONNECT: IC1.PIO0_6/USB_CONNECT/SCK0, R5.1
- removed net USB_D+: IC1.USB_DP, R2.1
- removed net USB_D-: IC1.USB_DM, R1.1
- removed net USB_FTOGGLE: IC1.PIO0_1/CLKOUT/CT32B0_MAT2/USB_FTOGGLE
- removed net USB_VBUS: IC1.PIO0_3/USB_VBUS, R8.2, R9.1
- removed net XTAL1: C2.2, IC1.XTALIN, Y1.CRYSTAL2
- removed net XTAL2: C1.2, IC1.XTALOUT, Y1.CRYSTAL1
- new net DW_EXTON: BOARD1.A0, IC1.EXTON
- new net DW_IRQ: BOARD1.B0, IC1.IRQ/GPIO8
- new net DW_RST: BOARD1.B1, IC1.!RST
- new net DW_WAKE: BOARD1.A1, IC1.WAKEUP
- new net I2C1_SCL: BOARD1.B6, CN_IMU.3
- new net I2C1_SDA: BOARD1.B7, CN_IMU.4
- new net LED_ACT: BOARD1.B3, R3.1
- new net LED_ERR: BOARD1.B4, R2.1
- new net LED_RXOK: IC1.GPIO0/RXOKLED, R7.1
- new net MPU_AD0: BOARD1.B9, CN_IMU.7
- new net N$7: C7.1, IC2.BYP
- new net SPI1_NSS: BOARD1.A4, IC1.!SPICS
- new net USART1_RX: BOARD1.A10, CN_USART1.3
- new net USART1_TX: BOARD1.A9, CN_USART1.2
- new net USART2_RX: BOARD1.A3, CN_USART2.3
- new net USART2_TX: BOARD1.A2, CN_USART2.2
- net +3V3: now also C1.1, C2.1, C3.1, C5.1, CN_IMU.1, IC1.VDD3V3, IC1.VDDAON; no longer C10.1, C11.1, C6.1, C8.1, C9.1, IC1.VDD1, IC1.VDD2, IC3.VDD3V3, IC3.VDDAON, IC4.!CS, IC4.AD0/SDO, IC4.RESV_VDDIO, IC4.VDD, IC4.VDDIO, JP1.1, Q1.E, R4.1, R6.1, R7.1
- net GND: now also ACT.C, BOARD1.GND, C1.2, C2.2, CN_IMU.10, CN_IMU.2, CN_USART1.1, CN_USART2.1, ERR.C, IC1.VSS, OK.C, SFD.C; no longer C1.1, C10.2, C11.2, C2.1, C8.2, C9.2, IC1.VSS1, IC1.VSS2, IC3.VSS, IC4.FSYNC, IC4.GND, IC4.RESV_GND, JP1.4, JTAG.3, JTAG.5, JTAG.9, R8.1, SYNC.GND@0, SYNC.GND@1, U$1.P$1, X1G$1.5, X1S.S1, X1S.S2, X1S.S3, X1S.S4, Y1.GND1, Y1.GND2
- net LED_RX: now also IC1.GPIO2/RXLED, R5.1; no longer IC3.GPIO2/RXLED, R11.2
- net LED_SFD: now also IC1.GPIO1/SFDLED, R6.1; no longer IC3.GPIO1/SFDLED
- net LED_SYS: now also BOARD1.B5, R1.1; no longer IC1.PIO0_18/RXD/CT32B0_MAT0, R13.2
- net LED_TX: now also IC1.GPIO3/TXLED, R4.1; no longer IC3.GPIO3/TXLED, R10.2
- net MPU_INT: now also BOARD1.B8, CN_IMU.8; no longer IC1.PIO0_21/CT16B1_MAT0/MOSI1, IC4.INT
- net N$1: now also RX.A; no longer Q1.B, R4.2
- net N$2: now also R4.2, TX.A; no longer Q1.C, R3.1
- net N$3: now also ACT.A, R3.2; no longer L1.2, X1G$1.1
- net N$4: now also ERR.A, R2.2; no longer IC1.PIO1_31, IC3.IRQ/GPIO8
- net N$5: now also SYS.A; no longer X1G$1.2
- net N$6: now also BOARD1.5V, C6.1, IC2.EN, IC2.IN; no longer IC3.SYNC, SYNC.SIGNAL
- net N$8: now also R6.2, SFD.A; no longer IC1.PIO0_7/CTS, IC3.!RST
- net N$9: now also OK.A, R7.2; no longer R10.1, TX.A
- net SPI1_MISO: now also BOARD1.A6, IC1.SPIMISO; no longer IC1.PIO1_21/DCD/MISO1, IC3.SPIMISO
- net SPI1_MOSI: now also BOARD1.A7, IC1.SPIMOSI; no longer IC1.PIO1_22/RI/MOSI1, IC3.SPIMOSI
- net SPI1_SCK: now also BOARD1.A5, IC1.SPICLK; no longer IC1.PIO1_20/DSR/SCK1, IC3.SPICLK
Other:
- moved on the sheet: C1, C2, C3, C4, C5, C6, C7, R1, R2, R3, R4, R5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
